File: CAN-Breakout.kicad_pcb (KiCad board)
At the start: 2 copper layers, 47.8 x 34 mm, 38 parts, among them J1 USB_C_Receptacle_USB2.0_16P, J2 DE9_Pins, J3 Conn_01x02_Pin, U1 ESP32-C6-MINI-1/U, U3 TLV70033_SOT23-5, U4 CDSOT23-T24CAN, U5 TCAN337, U6 USBLC6-2SC6

Commit message: rev1 comments + lakshay in person changes
Parts:
- removed C13: 10u, Capacitor_SMD:C_0603_1608Metric_Pad1.08x0.95mm_HandSolder
- removed JP1: CAN_RX_BKP_JMP, Connector_PinHeader_2.54mm:PinHeader_1x02_P2.54mm_Vertical
- removed JP2: CAN_TX_BKP_JMP, Connector_PinHeader_2.54mm:PinHeader_1x02_P2.54mm_Vertical
- removed TP6: CAN_RX_TP, Connector_PinHeader_2.54mm:PinHeader_1x01_P2.54mm_Vertical
- removed U6: USBLC6-2SC6, Package_TO_SOT_SMD:SOT-23-6
- added C3: 1u, Capacitor_SMD:C_0603_1608Metric_Pad1.08x0.95mm_HandSolder, F.Cu at (44.8, 47.1)
- added D10: BLE, Diode_SMD:D_0603_1608Metric_Pad1.05x0.95mm_HandSolder, F.Cu at (25.7, 60.2)
- added D5: 1N5819WS, Diode_SMD:D_SOD-323, F.Cu at (35.3, 65.1)
- added D6: CAN_FAULT_LED, Diode_SMD:D_0603_1608Metric_Pad1.05x0.95mm_HandSolder, F.Cu at (25.7, 49.9)
- added D7: CAN_TXD_LED, Diode_SMD:D_0603_1608Metric_Pad1.05x0.95mm_HandSolder, F.Cu at (25.7, 52.5)
- added D8: CAN_RXD_LED, Diode_SMD:D_0603_1608Metric_Pad1.05x0.95mm_HandSolder, F.Cu at (25.7, 55.0)
- added D9: HEARTBEAT, Diode_SMD:D_0603_1608Metric_Pad1.05x0.95mm_HandSolder, F.Cu at (25.7, 57.6)
- added J4: TERM_JMP, Connector_PinHeader_2.54mm:PinHeader_1x02_P2.54mm_Vertical, F.Cu at (65.8, 60.7)
- added J5: GPIO_BRKT, Connector_PinHeader_2.54mm:PinHeader_1x04_P2.54mm_Vertical, F.Cu at (62.3, 43.1)
- added R10: 10k, Resistor_SMD:R_0603_1608Metric_Pad0.98x0.95mm_HandSolder, F.Cu at (53.5, 54.6)
- added R11: 10k, Resistor_SMD:R_0603_1608Metric_Pad0.98x0.95mm_HandSolder, F.Cu at (53.5, 57.1)
- added R12: 160R, Resistor_SMD:R_0603_1608Metric_Pad0.98x0.95mm_HandSolder, F.Cu at (57.9, 42.0)
- added R13: 160R, Resistor_SMD:R_0603_1608Metric_Pad0.98x0.95mm_HandSolder, F.Cu at (57.9, 44.6)
- added R14: 160R, Resistor_SMD:R_0603_1608Metric_Pad0.98x0.95mm_HandSolder, F.Cu at (57.9, 47.1)
- added R15: 160R, Resistor_SMD:R_0603_1608Metric_Pad0.98x0.95mm_HandSolder, F.Cu at (57.9, 49.6)
- added R4: 160R, Resistor_SMD:R_0603_1608Metric_Pad0.98x0.95mm_HandSolder, F.Cu at (49.2, 57.1)
- added SW1: BOOT, Button_Switch_SMD:SW_SPST_B3S-1000, F.Cu at (62.0, 26.5)
- added TP1: CANH_TP, Connector_PinHeader_2.54mm:PinHeader_1x01_P2.54mm_Vertical, F.Cu at (61.2, 60.7)
- added TP2: CANL_TP, Connector_PinHeader_2.54mm:PinHeader_1x01_P2.54mm_Vertical, F.Cu at (61.2, 65.2)
- C11, C12, R1, R2, R7, R8: moved to F.Cu
- D3: value D_Zener -> SP0503BAHT; footprint Diode_SMD:D_0603_1608Metric_Pad1.05x0.95mm_HandSolder -> Package_TO_SOT_SMD:SOT-143
- F1: value 250mA Fuse -> 500mA Fuse; moved to F.Cu
- J3: value Conn_01x02_Pin -> UART_BRKT; footprint Connector_Molex:Molex_Nano-Fit_105309-xx02_1x02_P2.50mm_Vertical -> Connector_PinHeader_2.54mm:PinHeader_1x03_P2.54mm_Vertical
- TP3: value TP_CAN_L -> VBUS_TP; footprint Connector_PinHeader_2.54mm:PinHeader_1x01_P2.54mm_Vertical -> TestPoint:TestPoint_Pad_2.0x2.0mm
- TP4: value TP_CAN_H -> 5V_TP; footprint Connector_PinHeader_2.54mm:PinHeader_1x01_P2.54mm_Vertical -> TestPoint:TestPoint_Pad_2.0x2.0mm
- TP5: value CAN_TX_TP -> 3V3_TP; footprint Connector_PinHeader_2.54mm:PinHeader_1x01_P2.54mm_Vertical -> TestPoint:TestPoint_Pad_2.0x2.0mm
- moved J2 146.1 mm to (34.4, 25.6), turned to 0 degrees
- moved U5 123.8 mm to (30.5, 61.2), turned to 0 degrees
- moved D2 121.1 mm to (25.7, 44.7)
- moved U1 119.0 mm to (35.3, 49.9), turned to 0 degrees
- moved D1 118.1 mm to (25.7, 42.1), turned to 0 degrees
- moved U4 115.5 mm to (35.6, 61.4), turned to 0 degrees
- moved C8 114.8 mm to (44.8, 54.6), turned to 0 degrees
- moved SW_RST1 114.6 mm to (62.0, 35.0), turned to 0 degrees
- moved C9 114.2 mm to (44.8, 57.1), turned to 0 degrees
- moved C11 113.1 mm to (49.2, 44.6)
- moved TP5 110.4 mm to (66.7, 50.9)
- moved R7 110.2 mm to (53.5, 47.1), turned to 0 degrees
- moved C12 109.8 mm to (49.2, 47.1), turned to 0 degrees
- moved R9 108.9 mm to (53.5, 52.1)
- moved D4 107.8 mm to (25.7, 47.3)
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Connections:
- D3 pad 1: VBUS -> GND
- D3 pad 2: GND -> VBUS
- J1 pad A4: VBUS -> Net-(D5-A)
- J1 pad A6: Net-(J1-D+-PadA6) -> USB_DP
- J1 pad A7: Net-(J1-D--PadA7) -> USB_DN
- J1 pad A9: VBUS -> Net-(D5-A)
- J1 pad B4: VBUS -> Net-(D5-A)
- J1 pad B6: Net-(J1-D+-PadA6) -> USB_DP
- J1 pad B7: Net-(J1-D--PadA7) -> USB_DN
- J1 pad B9: VBUS -> Net-(D5-A)
- J2 pad 2: unconnected-(J2-Pad2) -> Net-(J4-Pin_2)
- J2 pad 3: CANH -> unconnected-(J2-Pad3)
- J2 pad 5: CANL -> unconnected-(J2-Pad5)
- J2 pad 7: unconnected-(J2-Pad7) -> Net-(U4-CAN_H)
- J3 pad 1: CANL -> U0TXD
- J3 pad 2: CANH -> U0RXD
- R9 pad 1: CANH -> Net-(J4-Pin_1)
- R9 pad 2: CANL -> Net-(U4-CAN_H)
- TP3 pad 1: CANL -> VBUS
- TP4 pad 1: CANH -> +5V
- TP5 pad 1: CAN_TXD -> +3V3
- U1 pad 10: unconnected-(U1-MTDI/GPIO5/ADC1_CH5-Pad10) -> CAN_RX_LED_PIN
- U1 pad 15: unconnected-(U1-MTCK/GPIO6/ADC1_CH6-Pad15) -> Net-(U1-MTCK/GPIO6/ADC1_CH6)
- U1 pad 16: unconnected-(U1-MTDO/GPIO7-Pad16) -> Net-(U1-MTDO/GPIO7)
- U1 pad 19: CAN_TXD_BKP1 -> Net-(J5-Pin_1)
- U1 pad 20: CAN_RXD_BKP1 -> Net-(J5-Pin_2)
- U1 pad 23: unconnected-(U1-GPIO9-Pad23) -> Net-(U1-GPIO9)
- U1 pad 24: unconnected-(U1-GPIO18-Pad24) -> Net-(J5-Pin_3)
- U1 pad 25: unconnected-(U1-GPIO19-Pad25) -> Net-(J5-Pin_4)
- U1 pad 26: CAN_TXD_BKP1 -> CAN_TXD
- U1 pad 27: CAN_RXD_BKP1 -> CAN_RXD
- U1 pad 29: unconnected-(U1-GPIO23-Pad29) -> Net-(U1-GPIO23)
- U1 pad 30: CAN_RXD -> U0RXD
- U1 pad 31: CAN_TXD -> U0TXD
- U1 pad 9: unconnected-(U1-MTMS/GPIO4/ADC1_CH4-Pad9) -> CAN_TX_LED_PIN
- U4 pad 1: CANH -> Net-(U4-CAN_H)
- U4 pad 2: CANL -> Net-(J4-Pin_2)
- U5 pad 3: Net-(U5-VCC) -> +3V3
- U5 pad 6: CANL -> Net-(J4-Pin_2)
- U5 pad 7: CANH -> Net-(U4-CAN_H)
Routing:
- net GND: track 102.7 -> 11.1 mm, vias 14 -> 0
- net CAN_TXD: track 42.7 -> 0.00 mm, vias 1 -> 0
- net CAN_RXD: track 40.5 -> 0.00 mm, vias 1 -> 0
- net CANH: track 27.3 -> 0.00 mm
- net CAN_TXD_BKP1: track 26.0 -> 0.00 mm
- net CANL: track 25.8 -> 0.00 mm, vias 2 -> 0
- net CAN_FAULT: track 25.3 -> 0.00 mm, vias 2 -> 0
- net VBUS: track 20.0 -> 0.00 mm, vias 2 -> 0
- net +5V: track 18.7 -> 0.00 mm, vias 2 -> 0
- net Net-(SW_RST1-B): track 13.4 -> 0.00 mm, vias 2 -> 0
- net USB_DN: track 11.9 -> 0.00 mm
- net CAN_RXD_BKP1: track 11.7 -> 0.00 mm
- net USB_DP: track 10.9 -> 0.00 mm
- net +3V3: track 10.4 -> 0.00 mm, vias 2 -> 0
- net Net-(J1-D+-PadA6): track 6.52 -> 0.00 mm
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- removed copper zone on F.Cu, net +3V3
- removed copper zone on B.Cu, net GND
Other:
- board outline removed
- board text removed: "3.3V"
- board text removed: "5.0V"
- board text removed: "CAN RX Backup"
- board text removed: "CAN TX Backup"
- board text removed: "CANH/CANL"
- board text removed: "CAN_RX CAN_TX"
- board text removed: "VBUS"

Commit message: layout v2
Parts:
- C3, R1, R2, R3, R4, R5, R6, R9, U4: moved to B.Cu
- F1 500mA: renamed from F1; moved to B.Cu
- moved J2 145.4 mm to (145.1, 119.9), turned to 180 degrees
- moved D7 129.1 mm to (128.2, 131.1), turned to 180 degrees
- moved D8 128.4 mm to (128.1, 132.6), turned to 180 degrees
- moved RESET 124.3 mm to (137.2, 133.9), turned to 180 degrees
- moved U5 123.9 mm to (137.2, 124.2)
- moved U4 122.8 mm to (141.5, 123.7), turned to -90 degrees
- moved C11 120.4 mm to (134.7, 129.4)
- moved C12 120.2 mm to (127.9, 137.9), turned to -90 degrees
- moved U1 119.1 mm to (116.0, 137.3), turned to 180 degrees
- moved C3 119.0 mm to (122.8, 136.9), turned to 180 degrees
- moved D6 118.7 mm to (103.7, 139.3)
- moved D2 117.7 mm to (120.4, 114.6)
- moved R7 115.4 mm to (131.1, 132.6), turned to -90 degrees
- moved BOOT 115.2 mm to (102.1, 134.4)
- moved C8 114.8 mm to (123.8, 137.9), turned to -90 degrees
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- renumbered SW1 to BOOT, TP1 to CANH, TP2 to CANL, SW_RST1 to RESET, TP5 to TP_3V3, TP4 to TP_5V, TP3 to TP_VBUS
Routing:
- net GND: track 11.1 -> 127.3 mm, vias 0 -> 32
- net +3V3: track 0.00 -> 59.5 mm, vias 0 -> 6
- net CAN_FAULT: track 0.00 -> 35.2 mm, vias 0 -> 2
- net CAN_TXD: track 0.00 -> 33.7 mm, vias 0 -> 4
- net CAN_RXD: track 0.00 -> 31.8 mm, vias 0 -> 4
- net USB_DN: track 0.00 -> 28.4 mm
- net USB_DP: track 0.00 -> 26.5 mm
- net Net-(U4-CAN_H): track 0.00 -> 25.0 mm, vias 0 -> 1
- net Net-(J5-Pin_4): track 0.00 -> 23.1 mm, vias 0 -> 2
- net Net-(J5-Pin_1): track 0.00 -> 20.2 mm, vias 0 -> 4
- net Net-(J5-Pin_3): track 0.00 -> 20.1 mm, vias 0 -> 2
- net Net-(J4-Pin_2): track 0.00 -> 20.0 mm, vias 0 -> 1
- net Net-(J5-Pin_2): track 0.00 -> 19.5 mm, vias 0 -> 4
- net +5V: track 0.00 -> 18.7 mm, vias 0 -> 1
- net U0TXD: track 0.00 -> 16.6 mm
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- added copper zone on B.Cu, net GND
Other:
- board outline added: 67 x 33.4 mm
- board text added: "BLUETOOTH"
- board text added: "CAN FLT"
- board text added: "CAN RX"
- board text added: "CAN TX"
- board text added: "GND RX TX"
- board text added: "HEARTBEAT"
- board text added: "TERM_JMP"
